File: circuit/Stingray.brd (EAGLE design)
At the start: 45.7 x 50.8 mm, 14 parts, among them IC1 4052N, IC2 4052N, K1 5200, K3 PN87520-S, M1 ARDUINO-NANO-3.0

Commit message: added files via upload
Parts:
- added R6, R7, R8: 10k, rcl:0204/7
- added X2: (no value), con-yamaichi:MDIN06SS
Connections:
- removed net TXD/SPARE: M1.J1.1
- new net PS2CLK: M1.J1.1, R6.2, X2.5
- new net PS2DAT: M1.J1.2, R7.2, X2.1
- net +5V: now also R6.1, R7.1, R8.2, X2.4
- net DETECT: now also M1.J2.6, R8.1; no longer M1.J1.2
- net GND: now also X2.3
Routing:
- net DETECT: track 61.6 -> 23.6 mm
- net PS2DAT: track 0.00 -> 31.2 mm
- net +5V: track 76.9 -> 104.6 mm
- net PS2CLK: track 0.00 -> 24.6 mm
- net GND: track 0.00 -> 6.35 mm
- net POTX1: track 20.6 -> 15.3 mm
- net VAC: track 29.1 -> 29.9 mm

Commit message: Alpha release, Joystick control seems fine, keyboard emulation to be tested.
Connections:
- net BOTTOM: now also K1.13, M1.J1.6; no longer K1.14, M1.J1.5
- net TOP: now also K1.14, M1.J1.5; no longer K1.13, M1.J1.6
Routing:
- net TOP: track 12.5 -> 11.3 mm
- net BOTTOM: track 11.3 -> 12.5 mm
Changed lines of the file:
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@@
 <layer number="49" name="Reference" color="7" fill="1" visible="no" active="yes"/>
 <layer number="50" name="dxf" color="7" fill="1" visible="no" active="no"/>
-<layer number="51" name="tDocu" color="7" fill="1" visible="no" active="yes"/>
+<layer number="51" name="tDocu" color="7" fill="1" visible="yes" active="yes"/>
 <layer number="52" name="bDocu" color="7" fill="1" visible="no" active="yes"/>
 <layer number="53" name="tGND_GNDA" color="7" fill="9" visible="no" active="no"/>
@@
 <wire x1="18.415" y1="43.18" x2="16.51" y2="43.18" width="0.3048" layer="1"/>
 </signal>
-<signal name="BOTTOM">
+<signal name="TOP">
 <contactref element="K1" pad="14"/>
 <contactref element="M1" pad="J1.5"/>
@@
 <wire x1="7.3025" y1="30.48" x2="12.7" y2="30.48" width="0.3048" layer="16"/>
 </signal>
-<signal name="TOP">
+<signal name="BOTTOM">
 <contactref element="K1" pad="13"/>
 <contactref element="M1" pad="J1.6"/>
